Commit message: pr2 updates

File: urdf/pr2.urdf (robot description, URDF)
Before this commit: robot pr2, 82 links, 81 joints
Links:
- removed link bl_caster_l_wheel_link
- removed link bl_caster_r_wheel_link
- removed link bl_caster_rotation_link
- removed link br_caster_l_wheel_link
- removed link br_caster_r_wheel_link
- removed link br_caster_rotation_link
- removed link fl_caster_l_wheel_link
- removed link fl_caster_r_wheel_link
- removed link fl_caster_rotation_link
- removed link fr_caster_l_wheel_link
- removed link fr_caster_r_wheel_link
- removed link fr_caster_rotation_link
- removed link l_gripper_l_parallel_link
- removed link l_gripper_r_parallel_link
- removed link narrow_stereo_gazebo_l_stereo_camera_frame
- removed link narrow_stereo_gazebo_l_stereo_camera_optical_frame
- removed link narrow_stereo_gazebo_r_stereo_camera_frame
- removed link narrow_stereo_gazebo_r_stereo_camera_optical_frame
- removed link r_gripper_l_parallel_link
- removed link r_gripper_r_parallel_link
- removed link wide_stereo_gazebo_l_stereo_camera_frame
- removed link wide_stereo_gazebo_l_stereo_camera_optical_frame
- removed link wide_stereo_gazebo_r_stereo_camera_frame
- removed link wide_stereo_gazebo_r_stereo_camera_optical_frame
- added link base_bellow_link, mass 1.0; collision box size=0.05 0.37 0.3; visual box size=0.05 0.37 0.3
- added link l_gripper_motor_screw_link, mass 0.01
- added link l_gripper_motor_slider_link, mass 0.01
- added link l_torso_lift_side_plate_link, mass 0.1
- added link narrow_stereo_l_stereo_camera_frame, mass 0.01
- added link narrow_stereo_l_stereo_camera_optical_frame
- added link narrow_stereo_r_stereo_camera_frame, mass 0.01
- added link narrow_stereo_r_stereo_camera_optical_frame
- added link projector_wg6802418_child_frame, mass 0.01
- added link projector_wg6802418_frame, mass 0.01
- added link r_gripper_motor_screw_link, mass 0.01
- added link r_gripper_motor_slider_link, mass 0.01
- added link r_torso_lift_side_plate_link, mass 0.1
- added link torso_lift_motor_screw_link, mass 1.0
- added link wide_stereo_l_stereo_camera_frame, mass 0.01
- added link wide_stereo_l_stereo_camera_optical_frame
- added link wide_stereo_r_stereo_camera_frame, mass 0.01
- added link wide_stereo_r_stereo_camera_optical_frame
- link base_laser_link: geometry 
- link base_link: geometry collision mesh filename=package://pr2_description/meshes/base_v0/base_L.stl; visual mesh filename=package://pr2_description/meshes/base_v0/base.dae
- link double_stereo_link: geometry visual box size=0.02 0.12 0.05
- link head_pan_link: mass 1.611118 -> 6.339; geometry collision mesh filename=package://pr2_description/meshes/head_v0/head_pan_L.stl; visual mesh filename=package://pr2_description/meshes/head_v0/head_pan.dae
- link head_tilt_link: mass 1.749727 -> 4.479; geometry collision mesh filename=package://pr2_description/meshes/head_v0/head_tilt_L.stl; visual mesh filename=package://pr2_description/meshes/head_v0/head_tilt.dae
- link high_def_frame: geometry 
- link high_def_optical_frame: geometry 
- link imu_link: geometry 
- link l_elbow_flex_link: geometry collision mesh filename=package://pr2_description/meshes/upper_arm_v0/elbow_flex.stl; visual mesh filename=package://pr2_description/meshes/upper_arm_v0/elbow_flex.dae
- link l_forearm_cam_frame: geometry 
- link l_forearm_link: geometry collision mesh filename=package://pr2_description/meshes/forearm_v0/forearm.stl; visual mesh filename=package://pr2_description/meshes/forearm_v0/forearm.dae
- link l_gripper_l_finger_link: geometry collision mesh filename=package://pr2_description/meshes/gripper_v0/l_finger.stl; visual mesh filename=package://pr2_description/meshes/gripper_v0/l_finger.dae
- link l_gripper_l_finger_tip_link: geometry collision mesh filename=package://pr2_description/meshes/gripper_v0/l_finger_tip.stl; visual mesh filename=package://pr2_description/meshes/gripper_v0/l_finger_tip.dae
- link l_gripper_palm_link: geometry collision mesh filename=package://pr2_description/meshes/gripper_v0/gripper_palm.stl; visual mesh filename=package://pr2_description/meshes/gripper_v0/gripper_palm.dae
- link l_gripper_r_finger_link: geometry collision mesh filename=package://pr2_description/meshes/gripper_v0/l_finger.stl; visual mesh filename=package://pr2_description/meshes/gripper_v0/l_finger.dae
- link l_gripper_r_finger_tip_link: geometry collision mesh filename=package://pr2_description/meshes/gripper_v0/l_finger_tip.stl; visual mesh filename=package://pr2_description/meshes/gripper_v0/l_finger_tip.dae
- link l_shoulder_pan_link: geometry collision mesh filename=package://pr2_description/meshes/shoulder_v0/shoulder_pan.s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; visual mesh filename=package://pr2_description/meshes/shoulder_v0/shoulder_pan.d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
- link l_upper_arm_link: geometry collision mesh filename=package://pr2_description/meshes/upper_arm_v0/upper_arm.stl; visual mesh filename=package://pr2_description/meshes/upper_arm_v0/upper_arm.dae
- link l_wrist_flex_link: geometry collision mesh filename=package://pr2_description/meshes/forearm_v0/wrist_flex.stl; visual mesh filename=package://pr2_description/meshes/forearm_v0/wrist_flex.dae
- link laser_tilt_link: geometry 
- link laser_tilt_mount_link: mass 0.05 -> 0.591
- link narrow_stereo_link: geometry 
- link r_elbow_flex_link: geometry collision mesh filename=package://pr2_description/meshes/upper_arm_v0/elbow_flex.stl; visual mesh filename=package://pr2_description/meshes/upper_arm_v0/elbow_flex.dae
- link r_forearm_cam_frame: geometry 
- link r_forearm_link: geometry collision mesh filename=package://pr2_description/meshes/forearm_v0/forearm.stl; visual mesh filename=package://pr2_description/meshes/forearm_v0/forearm.dae
- link r_gripper_l_finger_link: geometry collision mesh filename=package://pr2_description/meshes/gripper_v0/l_finger.stl; visual mesh filename=package://pr2_description/meshes/gripper_v0/l_finger.dae
- link r_gripper_l_finger_tip_link: geometry collision mesh filename=package://pr2_description/meshes/gripper_v0/l_finger_tip.stl; visual mesh filename=package://pr2_description/meshes/gripper_v0/l_finger_tip.dae
- link r_gripper_palm_link: geometry collision mesh filename=package://pr2_description/meshes/gripper_v0/gripper_palm.stl; visual mesh filename=package://pr2_description/meshes/gripper_v0/gripper_palm.dae
- link r_gripper_r_finger_link: geometry collision mesh filename=package://pr2_description/meshes/gripper_v0/l_finger.stl; visual mesh filename=package://pr2_description/meshes/gripper_v0/l_finger.dae
- link r_gripper_r_finger_tip_link: geometry collision mesh filename=package://pr2_description/meshes/gripper_v0/l_finger_tip.stl; visual mesh filename=package://pr2_description/meshes/gripper_v0/l_finger_tip.dae
- link r_shoulder_pan_link: geometry collision mesh filename=package://pr2_description/meshes/shoulder_v0/shoulder_pan.s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; visual mesh filename=package://pr2_description/meshes/shoulder_v0/shoulder_pan.d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
- link r_upper_arm_link: geometry collision mesh filename=package://pr2_description/meshes/upper_arm_v0/upper_arm.stl; visual mesh filename=package://pr2_description/meshes/upper_arm_v0/upper_arm.dae
- link r_wrist_flex_link: geometry collision mesh filename=package://pr2_description/meshes/forearm_v0/wrist_flex.stl; visual mesh filename=package://pr2_description/meshes/forearm_v0/wrist_flex.dae
- link sensor_mount_link: geometry visual box size=0.01 0.01 0.01
- link torso_lift_link: geometry collision mesh filename=package://pr2_description/meshes/torso_v0/torso_lift_L.stl; visual mesh filename=package://pr2_description/meshes/torso_v0/torso_lift.dae
- link wide_stereo_link: geometry 
Joints:
- removed joint bl_caster_l_wheel_joint
- removed joint bl_caster_r_wheel_joint
- removed joint bl_caster_rotation_joint
- removed joint br_caster_l_wheel_joint
- removed joint br_caster_r_wheel_joint
- removed joint br_caster_rotation_joint
- removed joint fl_caster_l_wheel_joint
- removed joint fl_caster_r_wheel_joint
- removed joint fl_caster_rotation_joint
- removed joint fr_caster_l_wheel_joint
- removed joint fr_caster_r_wheel_joint
- removed joint fr_caster_rotation_joint
- removed joint l_gripper_l_parallel_root_joint
- removed joint l_gripper_r_parallel_root_joint
- removed joint narrow_stereo_gazebo_l_stereo_camera_frame_joint
- removed joint narrow_stereo_gazebo_l_stereo_camera_optical_frame_joint
- removed joint narrow_stereo_gazebo_r_stereo_camera_frame_joint
- removed joint narrow_stereo_gazebo_r_stereo_camera_optical_frame_joint
- removed joint r_gripper_l_parallel_root_joint
- removed joint r_gripper_r_parallel_root_joint
- removed joint wide_stereo_gazebo_l_stereo_camera_frame_joint
- removed joint wide_stereo_gazebo_l_stereo_camera_optical_frame_joint
- removed joint wide_stereo_gazebo_r_stereo_camera_frame_joint
- removed joint wide_stereo_gazebo_r_stereo_camera_optical_frame_joint
- added joint base_bellow_joint: type fixed, parent base_link, child base_bellow_link, origin xyz=-0.29 0 0.8 rpy=0 0 0
- added joint l_gripper_motor_screw_joint: type continuous, parent l_gripper_motor_slider_link, child l_gripper_motor_screw_link, origin xyz=0.0 0 0 rpy=0 0 0, axis 0 1 0
- added joint l_gripper_motor_slider_joint: type prismatic, parent l_gripper_palm_link, child l_gripper_motor_slider_link, origin xyz=0.16828 0 0 rpy=0 0 0, axis 1 0 0, limit lower=-0.1 upper=0.1 effort=1000.0 velocity=0.2
- added joint l_torso_lift_side_plate_joint: type fixed, parent torso_lift_link, child l_torso_lift_side_plate_link, origin xyz=0.0535 0.209285 0.176625
- added joint narrow_stereo_l_stereo_camera_frame_joint: type fixed, parent narrow_stereo_link, child narrow_stereo_l_stereo_camera_frame, origin xyz=0 0 0 rpy=0 0 0
- added joint narrow_stereo_l_stereo_camera_optical_frame_joint: type fixed, parent narrow_stereo_l_stereo_camera_frame, child narrow_stereo_l_stereo_camera_optical_frame, origin xyz=0 0 0 rpy=-1.57079632679 0.0 -1.57079632679
- added joint narrow_stereo_r_stereo_camera_frame_joint: type fixed, parent narrow_stereo_l_stereo_camera_frame, child narrow_stereo_r_stereo_camera_frame, origin xyz=0.0 -0.09 0.0 rpy=0.0 0.0 0.0
- added joint narrow_stereo_r_stereo_camera_optical_frame_joint: type fixed, parent narrow_stereo_r_stereo_camera_frame, child narrow_stereo_r_stereo_camera_optical_frame, origin xyz=0 0 0 rpy=-1.57079632679 0.0 -1.57079632679
- added joint projector_wg6802418_child_frame_joint: type fixed, parent projector_wg6802418_frame, child projector_wg6802418_child_frame, origin xyz=0 0 0 rpy=0 -1.57079632679 0
- added joint projector_wg6802418_frame_joint: type fixed, parent head_plate_frame, child projector_wg6802418_frame, origin xyz=0.046457 0.110 0.0546 rpy=0 0 0
- added joint r_gripper_motor_screw_joint: type continuous, parent r_gripper_motor_slider_link, child r_gripper_motor_screw_link, origin xyz=0.0 0 0 rpy=0 0 0, axis 0 1 0
- added joint r_gripper_motor_slider_joint: type prismatic, parent r_gripper_palm_link, child r_gripper_motor_slider_link, origin xyz=0.16828 0 0 rpy=0 0 0, axis 1 0 0, limit lower=-0.1 upper=0.1 effort=1000.0 velocity=0.2
- added joint r_torso_lift_side_plate_joint: type fixed, parent torso_lift_link, child r_torso_lift_side_plate_link, origin xyz=0.0535  -0.209285 0.176625
- added joint torso_lift_motor_screw_joint: type continuous, parent base_link, child torso_lift_motor_screw_link, origin xyz=-0.15 0.0 0.7, axis 0 0 1
- added joint wide_stereo_l_stereo_camera_frame_joint: type fixed, parent wide_stereo_link, child wide_stereo_l_stereo_camera_frame, origin xyz=0 0 0 rpy=0 0 0
- added joint wide_stereo_l_stereo_camera_optical_frame_joint: type fixed, parent wide_stereo_l_stereo_camera_frame, child wide_stereo_l_stereo_camera_optical_frame, origin xyz=0 0 0 rpy=-1.57079632679 0.0 -1.57079632679
- added joint wide_stereo_r_stereo_camera_frame_joint: type fixed, parent wide_stereo_l_stereo_camera_frame, child wide_stereo_r_stereo_camera_frame, origin xyz=0.0 -0.09 0.0 rpy=0.0 0.0 0.0
- added joint wide_stereo_r_stereo_camera_optical_frame_joint: type fixed, parent wide_stereo_r_stereo_camera_frame, child wide_stereo_r_stereo_camera_optical_frame, origin xyz=0 0 0 rpy=-1.57079632679 0.0 -1.57079632679
- joint double_stereo_frame_joint: origin xyz=0.0 0.0 0.003 rpy=0 0 0 -> xyz=0.0 0.0 0.0 rpy=0 0 0
- joint head_tilt_joint: limit lower=-0.471238 upper=1.39626 effort=15 velocity=5 -> lower=-0.471238 upper=1.39626 effort=18 velocity=5
- joint high_def_frame_joint: origin xyz=0 -0.109 0.035 rpy=0 0 0 -> xyz=0.046457 -0.110 0.054600 rpy=0 0 0
- joint l_wrist_flex_joint: limit lower=-2.094 upper=0.0 effort=10 velocity=3.078 -> lower=-2.18 upper=0.0 effort=10 velocity=3.078
- joint narrow_stereo_frame_joint: origin xyz=0.0 0.06 0.0305 rpy=0.0   0.0   0.0 -> xyz=0.045 0.06 0.0501 rpy=0.0   0.0   0.0
- joint r_wrist_flex_joint: limit lower=-2.094 upper=0.0 effort=10 velocity=3.078 -> lower=-2.18 upper=0.0 effort=10 velocity=3.078
- joint torso_lift_joint: limit lower=0.0 upper=0.31 effort=10000 velocity=0.013 -> lower=0.0 upper=0.33 effort=10000 velocity=0.013
- joint wide_stereo_frame_joint: origin xyz=0.0 0.03 0.0305 rpy=0.0   0.0   0.0 -> xyz=0.045 0.03 0.0501 rpy=0.0   0.0   0.0
